Commit message: Updated robot urdf to include needle / remade moveit_config / secondary controller no longer launching for fake system.

File: ur5_moveit_config/config/ur5.urdf.xacro (robot description, xacro)
@@ -6,4 +6,3 @@
     <!-- Import control_xacro -->
     <xacro:include filename="ur5.ros2_control.xacro" />
-    <xacro:ur5_ros2_control name="FakeSystem" initial_positions_file="$(arg initial_positions_file)"/>
 </robot>

File: ur5_robot_description/urdf/ur5.xacro (robot description, xacro)
@@ -169,5 +169,24 @@
   </link>
   <link name="flange"/>
-  <link name="tool0"/>
+  <link name="needle">
+    <visual>
+      <geometry>
+        <cylinder length="0.10" radius="0.001"/>
+      </geometry>
+      <material name="metal">
+        <color rgba="0.8 0.8 0.8 1"/>
+      </material>
+    </visual>
+    <collision>
+      <geometry>
+        <cylinder length="0.15" radius="0.002"/>
+      </geometry>
+    </collision>
+    <inertial>
+      <mass value="0.005"/>
+      <origin xyz="0 0 0"/>
+      <inertia ixx="1e-6" ixy="0" ixz="0" iyy="1e-6" iyz="0" izz="1e-6"/>
+    </inertial>
+  </link>
   <joint name="world-base_link_fixed_joint" type="fixed">
     <origin rpy="0 0 0" xyz="0 0 0"/>
@@ -241,5 +260,5 @@
     <origin rpy="1.5707963267948966 0 1.5707963267948966" xyz="0 0 0"/>
     <parent link="flange"/>
-    <child link="tool0"/>
+    <child link="needle"/>
   </joint>
   <ros2_control name="GazeboSimSystem" type="system">
@@ -295,28 +314,3 @@
     </plugin>
   </gazebo>
-  <link name="needle">
-    <visual>
-      <geometry>
-        <cylinder length="0.10" radius="0.001"/>
-      </geometry>
-      <material name="metal">
-        <color rgba="0.8 0.8 0.8 1"/>
-      </material>
-    </visual>
-    <collision>
-      <geometry>
-        <cylinder length="0.15" radius="0.002"/>
-      </geometry>
-    </collision>
-    <inertial>
-      <mass value="0.005"/>
-      <origin xyz="0 0 0"/>
-      <inertia ixx="1e-6" ixy="0" ixz="0" iyy="1e-6" iyz="0" izz="1e-6"/>
-    </inertial>
-  </link>
-  <joint name="needle_fixed_joint" type="fixed">
-    <parent link="tool0"/>
-    <child link="needle"/>
-    <origin xyz="0 0 0" rpy="0 0 0"/>
-  </joint>
 </robot>
