Commit message: Fixing CMake file & updating urdf frames to ressemble original one.

File: ur5_robot_description/urdf/ur5.xacro (robot description, xacro)
@@ -12,4 +12,6 @@
    <xacro:arg name="force_abs_paths" default="false" />
   <link name="world"/>
+  <link name="base_link"/>
+  <link name="base"/>
   <link name="base_link_inertia">
     <visual>
@@ -168,6 +170,16 @@
   <link name="flange"/>
   <link name="tool0"/>
+  <joint name="world-base_link_fixed_joint" type="fixed">
+    <origin rpy="0 0 0" xyz="0 0 0"/>
+    <parent link="world"/>
+    <child link="base_link"/>
+  </joint>
+  <joint name="base_link-base_fixed_joint" type="fixed">
+    <origin rpy="0 0 3.141592653589793" xyz="0 0 0"/>
+    <parent link="base_link"/>
+    <child link="base"/>
+  </joint>
   <joint name="base_link-base_link_inertia" type="fixed">
-    <parent link="world"/>
+    <parent link="base_link"/>
     <child link="base_link_inertia"/>
     <origin rpy="0 0 3.141592653589793" xyz="0 0 0"/>
@@ -231,4 +243,58 @@
     <child link="tool0"/>
   </joint>
+  <transmission name="shoulder_pan_trans">
+    <type>transmission_interface/SimpleTransmission</type>
+    <joint name="shoulder_pan_joint">
+      <hardwareInterface>hardware_interface/PositionJointInterface</hardwareInterface>
+    </joint>
+    <actuator name="shoulder_pan_motor">
+      <mechanicalReduction>1</mechanicalReduction>
+    </actuator>
+  </transmission>
+  <transmission name="shoulder_lift_trans">
+    <type>transmission_interface/SimpleTransmission</type>
+    <joint name="shoulder_lift_joint">
+      <hardwareInterface>hardware_interface/PositionJointInterface</hardwareInterface>
+    </joint>
+    <actuator name="shoulder_lift_motor">
+      <mechanicalReduction>1</mechanicalReduction>
+    </actuator>
+  </transmission>
+  <transmission name="elbow_trans">
+    <type>transmission_interface/SimpleTransmission</type>
+    <joint name="elbow_joint">
+      <hardwareInterface>hardware_interface/PositionJointInterface</hardwareInterface>
+    </joint>
+    <actuator name="elbow_motor">
+      <mechanicalReduction>1</mechanicalReduction>
+    </actuator>
+  </transmission>
+  <transmission name="wrist_1_trans">
+    <type>transmission_interface/SimpleTransmission</type>
+    <joint name="wrist_1_joint">
+      <hardwareInterface>hardware_interface/PositionJointInterface</hardwareInterface>
+    </joint>
+    <actuator name="wrist_1_motor">
+      <mechanicalReduction>1</mechanicalReduction>
+    </actuator>
+  </transmission>
+  <transmission name="wrist_2_trans">
+    <type>transmission_interface/SimpleTransmission</type>
+    <joint name="wrist_2_joint">
+      <hardwareInterface>hardware_interface/PositionJointInterface</hardwareInterface>
+    </joint>
+    <actuator name="wrist_2_motor">
+      <mechanicalReduction>1</mechanicalReduction>
+    </actuator>
+  </transmission>
+  <transmission name="wrist_3_trans">
+    <type>transmission_interface/SimpleTransmission</type>
+    <joint name="wrist_3_joint">
+      <hardwareInterface>hardware_interface/PositionJointInterface</hardwareInterface>
+    </joint>
+    <actuator name="wrist_3_motor">
+      <mechanicalReduction>1</mechanicalReduction>
+    </actuator>
+  </transmission>
   <ros2_control name="GazeboSimSystem" type="system">
     <hardware>

Commit message: Busted moveitconfig.

File: ur5_robot_description/urdf/ur5.xacro (robot description, xacro)
@@ -243,58 +243,4 @@
     <child link="tool0"/>
   </joint>
-  <transmission name="shoulder_pan_trans">
-    <type>transmission_interface/SimpleTransmission</type>
-    <joint name="shoulder_pan_joint">
-      <hardwareInterface>hardware_interface/PositionJointInterface</hardwareInterface>
-    </joint>
-    <actuator name="shoulder_pan_motor">
-      <mechanicalReduction>1</mechanicalReduction>
-    </actuator>
-  </transmission>
-  <transmission name="shoulder_lift_trans">
-    <type>transmission_interface/SimpleTransmission</type>
-    <joint name="shoulder_lift_joint">
-      <hardwareInterface>hardware_interface/PositionJointInterface</hardwareInterface>
-    </joint>
-    <actuator name="shoulder_lift_motor">
-      <mechanicalReduction>1</mechanicalReduction>
-    </actuator>
-  </transmission>
-  <transmission name="elbow_trans">
-    <type>transmission_interface/SimpleTransmission</type>
-    <joint name="elbow_joint">
-      <hardwareInterface>hardware_interface/PositionJointInterface</hardwareInterface>
-    </joint>
-    <actuator name="elbow_motor">
-      <mechanicalReduction>1</mechanicalReduction>
-    </actuator>
-  </transmission>
-  <transmission name="wrist_1_trans">
-    <type>transmission_interface/SimpleTransmission</type>
-    <joint name="wrist_1_joint">
-      <hardwareInterface>hardware_interface/PositionJointInterface</hardwareInterface>
-    </joint>
-    <actuator name="wrist_1_motor">
-      <mechanicalReduction>1</mechanicalReduction>
-    </actuator>
-  </transmission>
-  <transmission name="wrist_2_trans">
-    <type>transmission_interface/SimpleTransmission</type>
-    <joint name="wrist_2_joint">
-      <hardwareInterface>hardware_interface/PositionJointInterface</hardwareInterface>
-    </joint>
-    <actuator name="wrist_2_motor">
-      <mechanicalReduction>1</mechanicalReduction>
-    </actuator>
-  </transmission>
-  <transmission name="wrist_3_trans">
-    <type>transmission_interface/SimpleTransmission</type>
-    <joint name="wrist_3_joint">
-      <hardwareInterface>hardware_interface/PositionJointInterface</hardwareInterface>
-    </joint>
-    <actuator name="wrist_3_motor">
-      <mechanicalReduction>1</mechanicalReduction>
-    </actuator>
-  </transmission>
   <ros2_control name="GazeboSimSystem" type="system">
     <hardware>

Commit message: needle

File: ur5_robot_description/urdf/ur5.xacro (robot description, xacro)
@@ -295,3 +295,28 @@
     </plugin>
   </gazebo>
+  <link name="needle">
+    <visual>
+      <geometry>
+        <cylinder length="0.15" radius="0.002"/>
+      </geometry>
+      <material name="metal">
+        <color rgba="0.8 0.8 0.8 1"/>
+      </material>
+    </visual>
+    <collision>
+      <geometry>
+        <cylinder length="0.15" radius="0.002"/>
+      </geometry>
+    </collision>
+    <inertial>
+      <mass value="0.005"/>
+      <origin xyz="0 0 0.075"/>
+      <inertia ixx="1e-6" ixy="0" ixz="0" iyy="1e-6" iyz="0" izz="1e-6"/>
+    </inertial>
+  </link>
+  <joint name="needle_fixed_joint" type="fixed">
+    <parent link="tool0"/>
+    <child link="needle"/>
+    <origin xyz="0 0 0.08" rpy="0 0 0"/>
+  </joint>
 </robot>

Commit message: remove gap from needle to eef

File: ur5_robot_description/urdf/ur5.xacro (robot description, xacro)
@@ -298,5 +298,5 @@
     <visual>
       <geometry>
-        <cylinder length="0.15" radius="0.002"/>
+        <cylinder length="0.10" radius="0.001"/>
       </geometry>
       <material name="metal">
@@ -311,5 +311,5 @@
     <inertial>
       <mass value="0.005"/>
-      <origin xyz="0 0 0.075"/>
+      <origin xyz="0 0 0"/>
       <inertia ixx="1e-6" ixy="0" ixz="0" iyy="1e-6" iyz="0" izz="1e-6"/>
     </inertial>
@@ -318,5 +318,5 @@
     <parent link="tool0"/>
     <child link="needle"/>
-    <origin xyz="0 0 0.08" rpy="0 0 0"/>
+    <origin xyz="0 0 0" rpy="0 0 0"/>
   </joint>
 </robot>

Commit message: pare down the collision meshes we're using. and move the UR5 Z-offset to the urdf instead of spawn

File: ur5_robot_description/urdf/ur5.xacro (robot description, xacro)
@@ -190,5 +190,5 @@
   </link>
   <joint name="world-base_link_fixed_joint" type="fixed">
-    <origin rpy="0 0 0" xyz="0 0 0"/>
+    <origin rpy="0 0 0" xyz="0 0 0.895"/>
     <parent link="world"/>
     <child link="base_link"/>

Commit message: Refactored launch file. Increased needle length, adjusted move_ur5 goal tolerances. Added all models meshes to collision planning scene.

File: ur5_robot_description/urdf/ur5.xacro (robot description, xacro)
@@ -172,5 +172,5 @@
     <visual>
       <geometry>
-        <cylinder length="0.10" radius="0.001"/>
+        <cylinder length="0.20" radius="0.001"/>
       </geometry>
       <material name="metal">
